Commit message: Here I have made changes and added some few xacro files

File: src/prac_robot_description/urdf/prac_robot.urdf.xacro (robot description, xacro)
@@ -1,85 +1,5 @@
 <?xml version="1.0"?>
 <robot name="prac_robot" xmlns:xacro="http://www.ros.org/wiki/xacro">
-    <material name="grey">
-        <color rgba="0.6 0.4 0.7 1" />
-    </material>
-    <material name="blue">
-        <color rgba="0 0.4 0.7 1" />
-    </material>
-    <material name="white">
-        <color rgba="1 1 1 1" />
-    </material>
-    <link name="base_footprint" />
-    <link name="base_link">
-        <visual>
-            <geometry>
-                <box size="0.6 0.4 0.2" />
-            </geometry>
-            <origin xyz="0 0 0.1" rpy="0 0 0" />
-            <material name="grey" />
-        </visual>
-    </link>
-    <link name="lidar_link">
-        <visual>
-            <geometry>
-                <cylinder radius="0.1" length="0.05" />
-            </geometry>
-            <origin xyz="0 0 0" rpy="0 0 0" />
-            <material name="white" />
-        </visual>
-    </link>
-     <link name="left_wheel">
-        <visual>
-            <geometry>
-                <cylinder radius="0.1" length="0.05" />
-            </geometry>
-            <origin xyz="0 0 0" rpy="1.57 0 0" />
-            <material name="white" />
-        </visual>
-    </link>
-    <link name="right_wheel">
-        <visual>
-            <geometry>
-                <cylinder radius="0.1" length="0.05" />
-            </geometry>
-            <origin xyz="0 0 0" rpy="1.57 0 0" />
-            <material name="white" />
-        </visual>
-    </link>
-    <link name="caster_wheel">
-        <visual>
-            <geometry>
-                <sphere radius="0.05" />
-            </geometry>
-            <origin xyz="0 0 0" rpy="0 0 0" />
-            <material name="white" />
-        </visual>
-    </link>
-    <joint name="base_joint" type="fixed">
-        <parent link="base_footprint" />
-        <child link="base_link" />
-        <origin xyz="0 0 0.1" rpy="0 0 0" />
-    </joint>
-    <joint name="base_lidar_joint" type="fixed">
-        <parent link="base_link" />
-        <child link="lidar_link" />
-        <origin xyz="0 0 0.225" rpy="0 0 0" />
-    </joint>
-    <joint name="base_left_joint" type="continuous">
-        <parent link="base_link" />
-        <child link="left_wheel" />
-        <origin xyz="-0.15 0.225 0" rpy="0 0 0" />
-        <axis xyz="0 1 0" />
-    </joint>
-    <joint name="base_right_joint" type="continuous">
-        <parent link="base_link" />
-        <child link="right_wheel" />
-        <origin xyz="-0.15 -0.225 0" rpy="0 0 0" />
-        <axis xyz="0 1 0" />
-    </joint>
-    <joint name="base_caster_joint" type="fixed">
-        <parent link="base_link" />
-        <child link="caster_wheel" />
-        <origin xyz="0.2 0 -0.05" rpy="0 0 0" />
-    </joint>
+    <xacro:include filename="properties.xacro" />
+    <xacro:include filename="mobile_base.xacro" />
 </robot>
