Commit message: I introduced inertial tags so that I can be able to simulate my visualized robot in Gazebo

File: src/prac_robot_description/urdf/mobile_base.xacro (robot description, xacro)
@@ -15,4 +15,6 @@
             <material name="grey" />
         </visual>
+        <xacro:box_inertia m="5.0" l="${base_length}" w="${base_width}" h="${base_height}"
+                           xyz="0 0 ${base_height / 2.0}" rpy="0 0 0" />
     </link>
     <link name="lidar_link">

File: src/prac_robot_description/urdf/properties.xacro (robot description, xacro)
@@ -10,3 +10,30 @@
         <color rgba="1 1 1 1" />
     </material>
+    <xacro:macro name="box_inertia" params="m l w h xyz rpy">
+        <inertial>
+            <origin xyz="${xyz}" rpy="${rpy}" />
+            <mass value="${m}" />
+            <inertia ixx="${(m/12) * (h*h + l*l)}" ixy="0" ixz="0"
+                     iyy="${(m/12) * (w*w + l*l)}" iyz="0"
+                     izz="${(m/12) * (w*w + h*h)}" />
+        </inertial>
+    </xacro:macro>
+    <xacro:macro name="wheel_inertia" params="m r h xyz rpy">
+        <inertial>
+            <origin xyz="${xyz}" rpy="${rpy}" />
+            <mass value="${m}" />
+            <inertia ixx="${(m/12) * (3*r*r + h*h)}" ixy="0" ixz="0"
+                     iyy="${(m/12) * (3*r*r + h*h)}" iyz="0"
+                     izz="${(m/12) * (r*r)}" />
+        </inertial>
+    </xacro:macro>
+    <xacro:macro name="caster inertia" params="m r xyz rpy">
+        <inertial>
+            <origin xyz="${xyz}" rpy="${rpy}" />
+            <mass value="${m}" />
+            <inertia ixx="${(2 * m/5) * (r*r)}" ixy="0" ixz="0"
+                     iyy="${(2 * m/5) * (r*r)}" iyz="0"
+                     izz="${(2 * m/5) * (r*r)}">
+        </inertial>
+    </xacro:macro>
 </robot>

Commit message: I have added all the required inertial and collision tags so that I can be able to visualize the robot in Gazebo

File: src/prac_robot_description/urdf/mobile_base.xacro (robot description, xacro)
@@ -15,4 +15,10 @@
             <material name="grey" />
         </visual>
+        <collision>
+            <geometry>
+                <box size="${base_length} ${base_width} ${base_height}" />
+            </geometry>
+            <origin xyz="0 0 ${base_height / 2.0}" rpy="0 0 0" />
+        </collision>
         <xacro:box_inertia m="5.0" l="${base_length}" w="${base_width}" h="${base_height}"
                            xyz="0 0 ${base_height / 2.0}" rpy="0 0 0" />
@@ -26,4 +32,12 @@
             <material name="white" />
         </visual>
+        <collision>
+            <geometry>
+                <cylinder radius="${wheel_radius}" length="${wheel_length}" />
+            </geometry>
+            <origin xyz="0 0 0" rpy="0 0 0" />
+        </collision>
+        <xacro:cylinder_inertia m="0.2" r="${wheel_radius}" h="${wheel_length}"
+                             xyz="0 0 0" rpy="0 0 0" />
     </link>
      <link name="left_wheel">
@@ -35,4 +49,12 @@
             <material name="white" />
         </visual>
+        <collision>
+            <geometry>
+                <cylinder radius="${wheel_radius}" length="${wheel_length}" />
+            </geometry>
+            <origin xyz="0 0 0" rpy="${pi / 2.0} 0 0" />
+        </collision>
+        <xacro:cylinder_inertia m="1.0" r="${wheel_radius}" h="${wheel_length}"
+                             xyz="0 0 0" rpy="${pi / 2.0} 0 0" />
     </link>
     <link name="right_wheel">
@@ -44,4 +66,12 @@
             <material name="white" />
         </visual>
+        <collision>
+            <geometry>
+                <cylinder radius="${wheel_radius}" length="${wheel_length}" />
+            </geometry>
+            <origin xyz="0 0 0" rpy="${pi / 2.0} 0 0" />
+        </collision>
+        <xacro:cylinder_inertia m="1.0" r="${wheel_radius}" h="${wheel_length}"
+                             xyz="0 0 0" rpy="${pi / 2.0} 0 0" />
     </link>
     <link name="caster_wheel">
@@ -53,4 +83,12 @@
             <material name="white" />
         </visual>
+        <collision>
+            <geometry>
+                <sphere radius="0.05" />
+            </geometry>
+            <origin xyz="0 0 0" rpy="0 0 0" />
+        </collision>
+        <xacro:sphere_inertia m="0.5" r="0.05"
+                              xyz="0 0 0" rpy="0 0 0" />
     </link>
     <joint name="base_joint" type="fixed">

File: src/prac_robot_description/urdf/properties.xacro (robot description, xacro)
@@ -19,5 +19,5 @@
         </inertial>
     </xacro:macro>
-    <xacro:macro name="wheel_inertia" params="m r h xyz rpy">
+    <xacro:macro name="lidar_inertia" params="m r h xyz rpy">
         <inertial>
             <origin xyz="${xyz}" rpy="${rpy}" />
@@ -28,5 +28,14 @@
         </inertial>
     </xacro:macro>
-    <xacro:macro name="caster inertia" params="m r xyz rpy">
+    <xacro:macro name="cylinder_inertia" params="m r h xyz rpy">
+        <inertial>
+            <origin xyz="${xyz}" rpy="${rpy}" />
+            <mass value="${m}" />
+            <inertia ixx="${(m/12) * (3*r*r + h*h)}" ixy="0" ixz="0"
+                     iyy="${(m/12) * (3*r*r + h*h)}" iyz="0"
+                     izz="${(m/12) * (r*r)}" />
+        </inertial>
+    </xacro:macro>
+    <xacro:macro name="sphere_inertia" params="m r xyz rpy">
         <inertial>
             <origin xyz="${xyz}" rpy="${rpy}" />
@@ -34,5 +43,5 @@
             <inertia ixx="${(2 * m/5) * (r*r)}" ixy="0" ixz="0"
                      iyy="${(2 * m/5) * (r*r)}" iyz="0"
-                     izz="${(2 * m/5) * (r*r)}">
+                     izz="${(2 * m/5) * (r*r)}" />
         </inertial>
     </xacro:macro>
