Commit message: I worked on a different launch file and a new environment for the robot, using the teleop twist I can now control my robot

File: my_robot-main/install/prac_robot_description/share/prac_robot_description/urdf/mobile_base.xacro (robot description, xacro)
@@ -1,148 +1 @@
-<?xml version="1.0"?>
-<robot xmlns:xacro="http://www.ros.org/wiki/xacro">
-    <xacro:property name="base_length" value="0.6" />
-    <xacro:property name="base_width" value="0.4" />
-    <xacro:property name="base_height" value="0.2" />
-    <xacro:property name="wheel_radius" value="0.1" />
-    <xacro:property name="wheel_length" value="0.05" />
-    <link name="base_footprint" />
-    <link name="base_link">
-        <visual>
-            <geometry>
-                <box size="${base_length} ${base_width} ${base_height}" />
-            </geometry>
-            <origin xyz="0 0 ${base_height / 2.0}" rpy="0 0 0" />
-            <material name="grey" />
-        </visual>
-        <collision>
-            <geometry>
-                <box size="${base_length} ${base_width} ${base_height}" />
-            </geometry>
-            <origin xyz="0 0 ${base_height / 2.0}" rpy="0 0 0" />
-        </collision>
-        <xacro:box_inertia m="5.0" l="${base_length}" w="${base_width}" h="${base_height}"
-                           xyz="0 0 ${base_height / 2.0}" rpy="0 0 0" />
-    </link>
-    <link name="lidar_link">
-        <visual>
-            <geometry>
-                <cylinder radius="${wheel_radius}" length="${wheel_length}" />
-            </geometry>
-            <origin xyz="0 0 0" rpy="0 0 0" />
-            <material name="white" />
-        </visual>
-        <collision>
-            <geometry>
-                <cylinder radius="${wheel_radius}" length="${wheel_length}" />
-            </geometry>
-            <origin xyz="0 0 0" rpy="0 0 0" />
-        </collision>
-        <xacro:cylinder_inertia m="0.2" r="${wheel_radius}" h="${wheel_length}"
-                             xyz="0 0 0" rpy="0 0 0" />
-    </link>
-     <link name="left_wheel">
-        <visual>
-            <geometry>
-                <cylinder radius="${wheel_radius}" length="${wheel_length}" />
-            </geometry>
-            <origin xyz="0 0 0" rpy="${pi / 2.0} 0 0" />
-            <material name="white" />
-        </visual>
-        <collision>
-            <geometry>
-                <cylinder radius="${wheel_radius}" length="${wheel_length}" />
-            </geometry>
-            <origin xyz="0 0 0" rpy="${pi / 2.0} 0 0" />
-        </collision>
-        <xacro:cylinder_inertia m="1.0" r="${wheel_radius}" h="${wheel_length}"
-                             xyz="0 0 0" rpy="${pi / 2.0} 0 0" />
-    </link>
-    <link name="right_wheel">
-        <visual>
-            <geometry>
-                <cylinder radius="${wheel_radius}" length="${wheel_length}" />
-            </geometry>
-            <origin xyz="0 0 0" rpy="${pi / 2.0} 0 0" />
-            <material name="white" />
-        </visual>
-        <collision>
-            <geometry>
-                <cylinder radius="${wheel_radius}" length="${wheel_length}" />
-            </geometry>
-            <origin xyz="0 0 0" rpy="${pi / 2.0} 0 0" />
-        </collision>
-        <xacro:cylinder_inertia m="1.0" r="${wheel_radius}" h="${wheel_length}"
-                             xyz="0 0 0" rpy="${pi / 2.0} 0 0" />
-    </link>
-    <link name="caster_wheel">
-        <visual>
-            <geometry>
-                <sphere radius="0.05" />
-            </geometry>
-            <origin xyz="0 0 0" rpy="0 0 0" />
-            <material name="white" />
-        </visual>
-        <collision>
-            <geometry>
-                <sphere radius="0.05" />
-            </geometry>
-            <origin xyz="0 0 0" rpy="0 0 0" />
-        </collision>
-        <xacro:sphere_inertia m="0.5" r="0.05"
-                              xyz="0 0 0" rpy="0 0 0" />
-    </link>
-    <joint name="base_joint" type="fixed">
-        <parent link="base_footprint" />
-        <child link="base_link" />
-        <origin xyz="0 0 ${base_height / 2.0}" rpy="0 0 0" />
-    </joint>
-    <joint name="base_lidar_joint" type="fixed">
-        <parent link="base_link" />
-        <child link="lidar_link" />
-        <origin xyz="0 0 ${base_height + (wheel_length / 2.0) }" rpy="0 0 0" />
-    </joint>
-    <joint name="base_left_joint" type="continuous">
-        <parent link="base_link" />
-        <child link="left_wheel" />
-        <origin xyz="${-base_length / 4.0} ${(base_width + wheel_length) / 2.0} 0" rpy="0 0 0" />
-        <axis xyz="0 1 0" />
-    </joint>
-    <joint name="base_right_joint" type="continuous">
-        <parent link="base_link" />
-        <child link="right_wheel" />
-        <origin xyz="${-base_length / 4.0} ${-(base_width + wheel_length) / 2.0} 0" rpy="0 0 0" />
-        <axis xyz="0 1 0" />
-    </joint>
-    <joint name="base_caster_joint" type="fixed">
-        <parent link="base_link" />
-        <child link="caster_wheel" />
-        <origin xyz="${base_length / 3.0} 0 -0.05" rpy="0 0 0" />
-    </joint>
-        <!-- ROS 2 Control -->
-    <ros2_control name="mobile_robot_hardware" type="system">
-        <hardware>
-            <plugin>gazebo_ros2_control/GazeboSystem</plugin>
-        </hardware>
-        <joint name="base_left_joint">
-            <command_interface name="velocity"/>
-            <state_interface name="position"/>
-            <state_interface name="velocity"/>
-        </joint>
-        <joint name="base_right_joint">
-            <command_interface name="velocity"/>
-            <state_interface name="position"/>
-            <state_interface name="velocity"/>
-        </joint>
-    </ros2_control>
-    <!-- Differential Drive Plugin -->
-        <gazebo>
-            <plugin filename="libgz-sim-diff-drive-system.so" name="gz::sim::systems::DiffDrive">
-                <left_joint>base_left_joint</left_joint>
-                <right_joint>base_right_joint</right_joint>
-                <wheel_separation>${base_width + wheel_length}</wheel_separation>
-                <wheel_radius>${wheel_radius}</wheel_radius>
-                <odom_publish_frequency>50.0</odom_publish_frequency>
-                <topic>cmd_vel</topic>
-            </plugin>
-        </gazebo>
-</robot>
+/home/nimrod/Desktop/my_robot/my_robot-main/src/prac_robot_description/urdf/mobile_base.xacro

File: my_robot-main/install/prac_robot_description/share/prac_robot_description/urdf/prac_robot.urdf.xacro (robot description, xacro)
@@ -1,5 +1 @@
-<?xml version="1.0"?>
-<robot name="prac_robot" xmlns:xacro="http://www.ros.org/wiki/xacro">
-    <xacro:include filename="properties.xacro" />
-    <xacro:include filename="mobile_base.xacro" />
-</robot>
+/home/nimrod/Desktop/my_robot/my_robot-main/src/prac_robot_description/urdf/prac_robot.urdf.xacro

File: my_robot-main/install/prac_robot_description/share/prac_robot_description/urdf/properties.xacro (robot description, xacro)
@@ -1,63 +1 @@
-<?xml version="1.0"?>
-<robot xmlns:xacro="http://www.ros.org/wiki/xacro">
-    <material name="grey">
-        <color rgba="0 0.4 0.7 1" />
-    </material>
-    <material name="blue">
-        <color rgba="0 0.4 0.7 1" />
-    </material>
-        <material name="white">
-        <color rgba="1 1 1 1" />
-    </material>
-    <xacro:macro name="box_inertia" params="m l w h xyz rpy">
-        <inertial>
-            <origin xyz="${xyz}" rpy="${rpy}" />
-            <mass value="${m}" />
-            <inertia ixx="${(m/12) * (h*h + l*l)}" ixy="0" ixz="0"
-                     iyy="${(m/12) * (w*w + l*l)}" iyz="0"
-                     izz="${(m/12) * (w*w + h*h)}" />
-        </inertial>
-    </xacro:macro>
-    <xacro:macro name="lidar_inertia" params="m r h xyz rpy">
-        <inertial>
-            <origin xyz="${xyz}" rpy="${rpy}" />
-            <mass value="${m}" />
-            <inertia ixx="${(m/12) * (3*r*r + h*h)}" ixy="0" ixz="0"
-                     iyy="${(m/12) * (3*r*r + h*h)}" iyz="0"
-                     izz="${(m/12) * (r*r)}" />
-        </inertial>
-    </xacro:macro>
-    <xacro:macro name="cylinder_inertia" params="m r h xyz rpy">
-        <inertial>
-            <origin xyz="${xyz}" rpy="${rpy}" />
-            <mass value="${m}" />
-            <inertia ixx="${(m/12) * (3*r*r + h*h)}" ixy="0" ixz="0"
-                     iyy="${(m/12) * (3*r*r + h*h)}" iyz="0"
-                     izz="${(m/12) * (r*r)}" />
-        </inertial>
-    </xacro:macro>
-    <xacro:macro name="sphere_inertia" params="m r xyz rpy">
-        <inertial>
-            <origin xyz="${xyz}" rpy="${rpy}" />
-            <mass value="${m}" />
-            <inertia ixx="${(2 * m/5) * (r*r)}" ixy="0" ixz="0"
-                     iyy="${(2 * m/5) * (r*r)}" iyz="0"
-                     izz="${(2 * m/5) * (r*r)}" />
-        </inertial>
-    </xacro:macro>
-        <!-- Gazebo Materials -->
-    <!-- Gazebo Physics for Base -->
-    <gazebo reference="base_link">
-        <mu1>0.2</mu1>
-        <mu2>0.2</mu2>
-    </gazebo>
-    <!-- Gazebo Physics for Wheels -->
-    <gazebo reference="left_wheel">
-        <mu1>1.0</mu1>
-        <mu2>1.0</mu2>
-    </gazebo>
-    <gazebo reference="right_wheel">
-        <mu1>1.0</mu1>
-        <mu2>1.0</mu2>
-    </gazebo>
-</robot>
+/home/nimrod/Desktop/my_robot/my_robot-main/src/prac_robot_description/urdf/properties.xacro

File: my_robot-main/src/prac_robot_description/urdf/prac_robot.urdf.xacro (robot description, xacro)
@@ -3,3 +3,4 @@
     <xacro:include filename="properties.xacro" />
     <xacro:include filename="mobile_base.xacro" />
+    <xacro:include filename="gazebo.xacro" />
 </robot>
