Commit message: Found the issue on my launch file and rectified the problem

File: my_robot-main/install/prac_robot_description/share/prac_robot_description/urdf/gazebo.xacro (robot description, xacro)
@@ -1 +1,74 @@
-/home/nimrod/Desktop/my_robot/my_robot-main/src/prac_robot_description/urdf/gazebo.xacro
+<?xml version="1.0"?>
+<robot>
+  <gazebo>
+    <plugin
+        filename="gz-sim-diff-drive-system"
+        name="gz::sim::systems::DiffDrive">
+        <!-- Topic for the command input -->
+        <topic>/cmd_vel</topic>
+        <!-- Wheel joints -->
+        <base_left_joint>left_wheel_joint</base_left_joint>
+        <base_right_joint>right_wheel_joint</base_right_joint>
+        <!-- Wheel parameters -->
+        <wheel_separation>0.3</wheel_separation>
+        <wheel_radius>0.1</wheel_radius>
+        <!-- Control gains and limits (optional) -->
+        <max_velocity>3.0</max_velocity>
+        <max_linear_acceleration>1</max_linear_acceleration>
+        <min_linear_acceleration>-1</min_linear_acceleration>
+        <max_angular_acceleration>2</max_angular_acceleration>
+        <min_angular_acceleration>-2</min_angular_acceleration>
+        <max_linear_velocity>0.5</max_linear_velocity>
+        <min_linear_velocity>-0.5</min_linear_velocity>
+        <max_angular_velocity>1</max_angular_velocity>
+        <min_angular_velocity>-1</min_angular_velocity>
+        <!-- Other parameters (optional) -->
+        <odom_topic>odom</odom_topic>
+        <tf_topic>tf</tf_topic>
+        <frame_id>odom</frame_id>
+        <child_frame_id>base_footprint</child_frame_id>
+        <odom_publish_frequency>30</odom_publish_frequency>
+    </plugin>
+    <plugin
+        filename="gz-sim-joint-state-publisher-system"
+        name="gz::sim::systems::JointStatePublisher">
+        <topic>joint_states</topic>
+        <joint_name>base_left_joint</joint_name>
+        <joint_name>base_right_joint</joint_name>
+    </plugin>
+        <plugin
+      filename="gz-sim-imu-system"
+      name="gz::sim::systems::Imu">
+    </plugin>
+  </gazebo>
+  <gazebo reference="camera_link">
+    <sensor name="camera" type="camera">
+      <camera>
+        <horizontal_fov>1.3962634</horizontal_fov>
+        <image>
+          <width>640</width>
+          <height>480</height>
+          <format>R8G8B8</format>
+        </image>
+        <clip>
+          <near>0.1</near>
+          <far>15</far>
+        </clip>
+        <noise>
+          <type>gaussian</type>
+          <!-- Noise is sampled independently per pixel on each frame.
+               That pixel's noise value is added to each of its color
+               channels, which at that point lie in the range [0,1]. -->
+          <mean>0.0</mean>
+          <stddev>0.007</stddev>
+        </noise>
+        <optical_frame_id>camera_link_optical</optical_frame_id>
+        <camera_info_topic>camera/camera_info</camera_info_topic>
+      </camera>
+      <always_on>1</always_on>
+      <update_rate>20</update_rate>
+      <visualize>true</visualize>
+      <topic>camera/image</topic>
+    </sensor>
+  </gazebo>
+</robot>

File: my_robot-main/install/prac_robot_description/share/prac_robot_description/urdf/mobile_base.xacro (robot description, xacro)
@@ -1 +1,166 @@
-/home/nimrod/Desktop/my_robot/my_robot-main/src/prac_robot_description/urdf/mobile_base.xacro
+<?xml version="1.0"?>
+<robot xmlns:xacro="http://www.ros.org/wiki/xacro">
+    <xacro:property name="base_length" value="0.6" />
+    <xacro:property name="base_width" value="0.4" />
+    <xacro:property name="base_height" value="0.2" />
+    <xacro:property name="wheel_radius" value="0.1" />
+    <xacro:property name="wheel_length" value="0.05" />
+    <link name="base_footprint" />
+    <link name="base_link">
+        <visual>
+            <geometry>
+                <box size="${base_length} ${base_width} ${base_height}" />
+            </geometry>
+            <origin xyz="0 0 ${base_height / 2.0}" rpy="0 0 0" />
+            <material name="grey" />
+        </visual>
+        <collision>
+            <geometry>
+                <box size="${base_length} ${base_width} ${base_height}" />
+            </geometry>
+            <origin xyz="0 0 ${base_height / 2.0}" rpy="0 0 0" />
+        </collision>
+        <xacro:box_inertia m="5.0" l="${base_length}" w="${base_width}" h="${base_height}"
+                           xyz="0 0 ${base_height / 2.0}" rpy="0 0 0" />
+    </link>
+    <link name="camera_link">
+        <visual>
+            <geometry>
+                <cylinder radius="${wheel_radius}" length="${wheel_length}" />
+            </geometry>
+            <origin xyz="0 0 0" rpy="0 0 0" />
+            <material name="white" />
+        </visual>
+        <collision>
+            <geometry>
+                <cylinder radius="${wheel_radius}" length="${wheel_length}" />
+            </geometry>
+            <origin xyz="0 0 0" rpy="0 0 0" />
+        </collision>
+        <xacro:cylinder_inertia m="0.2" r="${wheel_radius}" h="${wheel_length}"
+                             xyz="0 0 0" rpy="0 0 0" />
+    </link>
+     <link name="left_wheel">
+        <visual>
+            <geometry>
+                <cylinder radius="${wheel_radius}" length="${wheel_length}" />
+            </geometry>
+            <origin xyz="0 0 0" rpy="${pi / 2.0} 0 0" />
+            <material name="white" />
+        </visual>
+        <collision>
+            <geometry>
+                <cylinder radius="${wheel_radius}" length="${wheel_length}" />
+            </geometry>
+            <origin xyz="0 0 0" rpy="${pi / 2.0} 0 0" />
+        </collision>
+        <xacro:cylinder_inertia m="1.0" r="${wheel_radius}" h="${wheel_length}"
+                             xyz="0 0 0" rpy="${pi / 2.0} 0 0" />
+    </link>
+    <link name="right_wheel">
+        <visual>
+            <geometry>
+                <cylinder radius="${wheel_radius}" length="${wheel_length}" />
+            </geometry>
+            <origin xyz="0 0 0" rpy="${pi / 2.0} 0 0" />
+            <material name="white" />
+        </visual>
+        <collision>
+            <geometry>
+                <cylinder radius="${wheel_radius}" length="${wheel_length}" />
+            </geometry>
+            <origin xyz="0 0 0" rpy="${pi / 2.0} 0 0" />
+        </collision>
+        <xacro:cylinder_inertia m="1.0" r="${wheel_radius}" h="${wheel_length}"
+                             xyz="0 0 0" rpy="${pi / 2.0} 0 0" />
+    </link>
+    <link name="caster_wheel">
+        <visual>
+            <geometry>
+                <sphere radius="0.05" />
+            </geometry>
+            <origin xyz="0 0 0" rpy="0 0 0" />
+            <material name="white" />
+        </visual>
+        <collision>
+            <geometry>
+                <sphere radius="0.05" />
+            </geometry>
+            <origin xyz="0 0 0" rpy="0 0 0" />
+        </collision>
+        <xacro:sphere_inertia m="0.5" r="0.05"
+                              xyz="0 0 0" rpy="0 0 0" />
+    </link>
+    <joint name="base_joint" type="fixed">
+        <parent link="base_footprint" />
+        <child link="base_link" />
+        <origin xyz="0 0 ${base_height / 2.0}" rpy="0 0 0" />
+    </joint>
+    <joint name="base_camera_joint" type="fixed">
+        <parent link="base_link" />
+        <child link="camera_link" />
+        <origin xyz="0 0 ${base_height + (wheel_length / 2.0) }" rpy="0 0 0" />
+    </joint>
+    <gazebo reference="camera_link">
+        <material>Gazebo/Red</material>
+    </gazebo>
+    <joint type="fixed" name="camera_optical_joint">
+        <origin xyz="0 0 0" rpy="-1.5707 0 -1.5707"/>
+        <child link="camera_link_optical"/>
+        <parent link="camera_link"/>
+    </joint>
+    <link name="camera_link_optical">
+    </link>
+    <joint name="base_left_joint" type="continuous">
+        <parent link="base_link" />
+        <child link="left_wheel" />
+        <origin xyz="${-base_length / 4.0} ${(base_width + wheel_length) / 2.0} 0" rpy="0 0 0" />
+        <axis xyz="0 1 0" />
+    </joint>
+    <joint name="base_right_joint" type="continuous">
+        <parent link="base_link" />
+        <child link="right_wheel" />
+        <origin xyz="${-base_length / 4.0} ${-(base_width + wheel_length) / 2.0} 0" rpy="0 0 0" />
+        <axis xyz="0 1 0" />
+    </joint>
+    <joint name="base_caster_joint" type="fixed">
+        <parent link="base_link" />
+        <child link="caster_wheel" />
+        <origin xyz="${base_length / 3.0} 0 -0.05" rpy="0 0 0" />
+    </joint>
+      <!-- STEP 8 - IMU -->
+  <joint name="imu_joint" type="fixed">
+    <origin xyz="0 0 0" rpy="0 0 0" />
+    <parent link="base_link"/>
+    <child link="imu_link" />
+  </joint>
+  <link name="imu_link">
+  </link>
+        <!-- ROS 2 Control -->
+    <ros2_control name="mobile_robot_hardware" type="system">
+        <hardware>
+            <plugin>gazebo_ros2_control/GazeboSystem</plugin>
+        </hardware>
+        <joint name="base_left_joint">
+            <command_interface name="velocity"/>
+            <state_interface name="position"/>
+            <state_interface name="velocity"/>
+        </joint>
+        <joint name="base_right_joint">
+            <command_interface name="velocity"/>
+            <state_interface name="position"/>
+            <state_interface name="velocity"/>
+        </joint>
+    </ros2_control>
+    <!-- Differential Drive Plugin -->
+        <gazebo>
+            <plugin filename="libgz-sim-diff-drive-system.so" name="gz::sim::systems::DiffDrive">
+                <left_joint>base_left_joint</left_joint>
+                <right_joint>base_right_joint</right_joint>
+                <wheel_separation>${base_width + wheel_length}</wheel_separation>
+                <wheel_radius>${wheel_radius}</wheel_radius>
+                <odom_publish_frequency>50.0</odom_publish_frequency>
+                <topic>cmd_vel</topic>
+            </plugin>
+        </gazebo>
+</robot>

File: my_robot-main/install/prac_robot_description/share/prac_robot_description/urdf/prac_robot.urdf.xacro (robot description, xacro)
@@ -1 +1,6 @@
-/home/nimrod/Desktop/my_robot/my_robot-main/src/prac_robot_description/urdf/prac_robot.urdf.xacro
+<?xml version="1.0"?>
+<robot name="prac_robot" xmlns:xacro="http://www.ros.org/wiki/xacro">
+    <xacro:include filename="properties.xacro" />
+    <xacro:include filename="mobile_base.xacro" />
+    <xacro:include filename="gazebo.xacro" />
+</robot>

File: my_robot-main/install/prac_robot_description/share/prac_robot_description/urdf/properties.xacro (robot description, xacro)
@@ -1 +1,63 @@
-/home/nimrod/Desktop/my_robot/my_robot-main/src/prac_robot_description/urdf/properties.xacro
+<?xml version="1.0"?>
+<robot xmlns:xacro="http://www.ros.org/wiki/xacro">
+    <material name="grey">
+        <color rgba="0 0.4 0.7 1" />
+    </material>
+    <material name="blue">
+        <color rgba="0 0.4 0.7 1" />
+    </material>
+        <material name="white">
+        <color rgba="1 1 1 1" />
+    </material>
+    <xacro:macro name="box_inertia" params="m l w h xyz rpy">
+        <inertial>
+            <origin xyz="${xyz}" rpy="${rpy}" />
+            <mass value="${m}" />
+            <inertia ixx="${(m/12) * (h*h + l*l)}" ixy="0" ixz="0"
+                     iyy="${(m/12) * (w*w + l*l)}" iyz="0"
+                     izz="${(m/12) * (w*w + h*h)}" />
+        </inertial>
+    </xacro:macro>
+    <xacro:macro name="lidar_inertia" params="m r h xyz rpy">
+        <inertial>
+            <origin xyz="${xyz}" rpy="${rpy}" />
+            <mass value="${m}" />
+            <inertia ixx="${(m/12) * (3*r*r + h*h)}" ixy="0" ixz="0"
+                     iyy="${(m/12) * (3*r*r + h*h)}" iyz="0"
+                     izz="${(m/12) * (r*r)}" />
+        </inertial>
+    </xacro:macro>
+    <xacro:macro name="cylinder_inertia" params="m r h xyz rpy">
+        <inertial>
+            <origin xyz="${xyz}" rpy="${rpy}" />
+            <mass value="${m}" />
+            <inertia ixx="${(m/12) * (3*r*r + h*h)}" ixy="0" ixz="0"
+                     iyy="${(m/12) * (3*r*r + h*h)}" iyz="0"
+                     izz="${(m/12) * (r*r)}" />
+        </inertial>
+    </xacro:macro>
+    <xacro:macro name="sphere_inertia" params="m r xyz rpy">
+        <inertial>
+            <origin xyz="${xyz}" rpy="${rpy}" />
+            <mass value="${m}" />
+            <inertia ixx="${(2 * m/5) * (r*r)}" ixy="0" ixz="0"
+                     iyy="${(2 * m/5) * (r*r)}" iyz="0"
+                     izz="${(2 * m/5) * (r*r)}" />
+        </inertial>
+    </xacro:macro>
+        <!-- Gazebo Materials -->
+    <!-- Gazebo Physics for Base -->
+    <gazebo reference="base_link">
+        <mu1>0.2</mu1>
+        <mu2>0.2</mu2>
+    </gazebo>
+    <!-- Gazebo Physics for Wheels -->
+    <gazebo reference="left_wheel">
+        <mu1>1.0</mu1>
+        <mu2>1.0</mu2>
+    </gazebo>
+    <gazebo reference="right_wheel">
+        <mu1>1.0</mu1>
+        <mu2>1.0</mu2>
+    </gazebo>
+</robot>

File: my_robot-main/src/prac_robot_description/urdf/gazebo.xacro (robot description, xacro)
@@ -37,4 +37,38 @@
         <joint_name>base_right_joint</joint_name>
     </plugin>
+        <plugin
+      filename="gz-sim-imu-system"
+      name="gz::sim::systems::Imu">
+    </plugin>
+  </gazebo>
+  <gazebo reference="camera_link">
+    <sensor name="camera" type="camera">
+      <camera>
+        <horizontal_fov>1.3962634</horizontal_fov>
+        <image>
+          <width>640</width>
+          <height>480</height>
+          <format>R8G8B8</format>
+        </image>
+        <clip>
+          <near>0.1</near>
+          <far>15</far>
+        </clip>
+        <noise>
+          <type>gaussian</type>
+          <!-- Noise is sampled independently per pixel on each frame.
+               That pixel's noise value is added to each of its color
+               channels, which at that point lie in the range [0,1]. -->
+          <mean>0.0</mean>
+          <stddev>0.007</stddev>
+        </noise>
+        <optical_frame_id>camera_link_optical</optical_frame_id>
+        <camera_info_topic>camera/camera_info</camera_info_topic>
+      </camera>
+      <always_on>1</always_on>
+      <update_rate>20</update_rate>
+      <visualize>true</visualize>
+      <topic>camera/image</topic>
+    </sensor>
   </gazebo>
 </robot>

File: my_robot-main/src/prac_robot_description/urdf/mobile_base.xacro (robot description, xacro)
@@ -24,5 +24,5 @@
                            xyz="0 0 ${base_height / 2.0}" rpy="0 0 0" />
     </link>
-    <link name="lidar_link">
+    <link name="camera_link">
         <visual>
             <geometry>
@@ -97,9 +97,19 @@
         <origin xyz="0 0 ${base_height / 2.0}" rpy="0 0 0" />
     </joint>
-    <joint name="base_lidar_joint" type="fixed">
+    <joint name="base_camera_joint" type="fixed">
         <parent link="base_link" />
-        <child link="lidar_link" />
+        <child link="camera_link" />
         <origin xyz="0 0 ${base_height + (wheel_length / 2.0) }" rpy="0 0 0" />
     </joint>
+    <gazebo reference="camera_link">
+        <material>Gazebo/Red</material>
+    </gazebo>
+    <joint type="fixed" name="camera_optical_joint">
+        <origin xyz="0 0 0" rpy="-1.5707 0 -1.5707"/>
+        <child link="camera_link_optical"/>
+        <parent link="camera_link"/>
+    </joint>
+    <link name="camera_link_optical">
+    </link>
     <joint name="base_left_joint" type="continuous">
         <parent link="base_link" />
@@ -119,4 +129,12 @@
         <origin xyz="${base_length / 3.0} 0 -0.05" rpy="0 0 0" />
     </joint>
+      <!-- STEP 8 - IMU -->
+  <joint name="imu_joint" type="fixed">
+    <origin xyz="0 0 0" rpy="0 0 0" />
+    <parent link="base_link"/>
+    <child link="imu_link" />
+  </joint>
+  <link name="imu_link">
+  </link>
         <!-- ROS 2 Control -->
     <ros2_control name="mobile_robot_hardware" type="system">
